Commit message: First joint

File: src/arduinobot_description/urdf/arduinobot.urdf.xacro (robot description, xacro)
@@ -97,122 +97,4 @@
         </collision>
     </link>
-    <!-- Second Joint & First Link -->
-    <joint name ="joint_2" type="revolute">
-        <parent link="base_plate"/>
-        <child link = "forward_drive_arm"/>
-        <origin xyz="-0.02 0 0.35"/>
-        <axis xyz="1 0 0"/>
-        <limit lower="-${PI / 2}" upper="${PI / 2}"
-                effort="${effort}" velocity="${velocity}"/>
-    </joint>
-    <link name="forward_drive_arm">
-        <xacro:default_inertial mass="0.1"/>
-        <visual>
-            <origin rpy=" 0 -${PI / 2} ${PI / 2}" xyz="0.19 0.06 -0.08"/>
-            <geometry>
-                <mesh filename="package://arduinobot_description/meshes/forward_drive_arm.STL" scale="0.01 0.01 0.01"/>
-            </geometry>
-        </visual>
-        <collision>
-            <origin rpy=" 0 -${PI / 2} ${PI / 2}" xyz="0.19 0.06 -0.08"/>
-            <geometry>
-                <mesh filename="package://arduinobot_description/meshes/forward_drive_arm.STL" scale="0.01 0.01 0.01"/>
-            </geometry>
-        </collision>
-    </link>
-<!-- Third Joint & Link  -->
-    <joint name ="joint_3" type="revolute">
-        <parent link="forward_drive_arm"/>
-        <child link = "horizontal_arm"/>
-        <origin xyz="0 0 0.8"/>
-        <axis xyz="1 0 0"/>
-        <limit lower="-${PI / 2}" upper="${PI / 2}"
-               effort="${effort}" velocity="${velocity}"/>
-    </joint>
-    <link name="horizontal_arm">
-        <xacro:default_inertial mass="0.1"/>
-        <visual>
-            <origin rpy="${PI / 2} 0 ${PI / 2}" xyz="-0.03 -0.4 -0.06"/>
-            <geometry>
-                <mesh filename="package://arduinobot_description/meshes/horizontal_arm.STL" scale="0.01 0.01 0.01"/>
-            </geometry>
-        </visual>
-        <collision>
-            <origin rpy="${PI / 2} 0 ${PI / 2}" xyz="-0.03 -0.4 -0.06"/>
-            <geometry>
-                <mesh filename="package://arduinobot_description/meshes/horizontal_arm.STL" scale="0.01 0.01 0.01"/>
-            </geometry>
-        </collision>
-    </link>
-    <!-- Forth Joint & Link  -->
-    <joint name ="horizontal_arm_to_claw_support" type="fixed">
-        <parent link="horizontal_arm"/>
-        <child link = "claw_support"/>
-        <origin xyz="0 0.82 0"/>
-    </joint>
-    <link name="claw_support">
-        <xacro:default_inertial mass="0.05"/>
-        <visual>
-            <origin rpy="0 0 ${PI / 2}" xyz="0.0 -0.05 -0.15"/>
-            <geometry>
-                <mesh filename="package://arduinobot_description/meshes/claw_support.STL" scale="0.01 0.01 0.01"/>
-            </geometry>
-        </visual>
-        <collision>
-            <origin rpy="0 0 ${PI / 2}" xyz="0 -0.05 -0.15"/>
-            <geometry>
-                <mesh filename="package://arduinobot_description/meshes/claw_support.STL" scale="0.01 0.01 0.01"/>
-            </geometry>
-        </collision>
-    </link>
-    <!-- Fivth Joint & Link  -->
-    <joint name ="joint_4" type="revolute">
-        <parent link="claw_support"/>
-        <child link = "gripper_right"/>
-        <origin xyz="-0.04 0.13 -0.1"/>
-        <axis xyz="0 0 1"/>
-        <limit lower="-${PI / 2}" upper="0.0"
-               effort="${effort}" velocity="${velocity}"/>
-    </joint>
-    <link name="gripper_right">
-        <xacro:default_inertial mass="0.01"/>
-        <visual>
-            <origin rpy="0 0 -${PI / 2}" xyz="-0.1 0.50 -0.1"/>
-            <geometry>
-                <mesh filename="package://arduinobot_description/meshes/right_finger.STL" scale="0.01 0.01 0.01"/>
-            </geometry>
-        </visual>
-        <collision>
-            <origin rpy="0 0 -${PI / 2}" xyz="-0.1 0.50 -0.1"/>
-            <geometry>
-                <mesh filename="package://arduinobot_description/meshes/right_finger.STL" scale="0.01 0.01 0.01"/>
-            </geometry>
-        </collision>
-    </link>
-    <!-- Sixth Joint & Link  -->
-    <joint name ="joint_5" type="revolute">
-        <parent link="claw_support"/>
-        <child link = "gripper_left"/>
-        <origin xyz="-0.22 0.13 -0.1"/>
-        <axis xyz="0 0 1"/>
-        <limit lower="0.0" upper="${PI / 2}"
-               effort="${effort}" velocity="${velocity}"/>
-        <mimic joint="joint_4" multiplier="-1"/>
-    </joint>
-    <link name="gripper_left">
-        <xacro:default_inertial mass="0.01"/>
-        <visual>
-            <origin rpy="0 0 -${PI / 2}" xyz="-0.04 0.50 -0.1"/>
-            <geometry>
-                <mesh filename="package://arduinobot_description/meshes/left_finger.STL" scale="0.01 0.01 0.01"/>
-            </geometry>
-        </visual>
-        <collision>
-            <origin rpy="0 0 -${PI / 2}" xyz="-0.04 0.50 -0.1"/>
-            <geometry>
-                <mesh filename="package://arduinobot_description/meshes/left_finger.STL" scale="0.01 0.01 0.01"/>
-            </geometry>
-        </collision>
-    </link>
     <gazebo reference="rgb_camera">
         <sensor type="camera" name="rgb_camera">

File: src/arduinobot_description/urdf/arduinobot_ros2_control.xacro (robot description, xacro)
@@ -14,33 +14,4 @@
             <state_interface name="position"/>
         </joint>
-        <joint name="joint_2">
-            <command_interface name="position">
-                <param name="min">-${PI/2}</param>
-                <param name="max">${PI/2}</param>
-            </command_interface>
-            <state_interface name="position"/>
-        </joint>
-        <joint name="joint_3">
-            <command_interface name="position">
-                <param name="min">-${PI/2}</param>
-                <param name="max">${PI/2}</param>
-            </command_interface>
-            <state_interface name="position"/>
-        </joint>
-        <joint name="joint_4">
-            <command_interface name="position">
-                <param name="min">-${PI/2}</param>
-                <param name="max">0.0</param>
-            </command_interface>
-            <state_interface name="position"/>
-        </joint>
-        <joint name="joint_5">
-            <param name="mimic">joint_4</param>
-            <param name="multiplier">-1</param>
-            <command_interface name="position">
-            <param name="min">0.0</param>
-            <param name="max">${PI / 2}</param>
-            </command_interface>
-        </joint>
     </ros2_control>
 </robot>
